File: 3PDT Board.brd (EAGLE design)
At the start: 23.8 x 22.2 mm, 10 parts, among them SW2 3PDT

Commit message: Fixed ground connections so jack grounds actually connect to ground!
Connections:
- net GND: now also JIG.1, JOG.1
Changed lines of the file:
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@@
 </polygon>
 <contactref element="SW2" pad="B2"/>
+<contactref element="JOG" pad="1"/>
+<contactref element="JIG" pad="1"/>
 </signal>
 <signal name="IN">

Commit message: Fixed circuit and made panel
Parts:
- removed IN: IN(T), mb_supply:SQUARE
- removed JOUT, LED: (no value), mb_supply:SQUARE
- removed OUT: OUT(T), mb_supply:SQUARE
- added D1: 1N4001, mb_diodes:DO41-3
- added JOT: (no value), mb_supply:SQUARE
- added U$1: BOARDLINK, xc_library:BOARDLINK
- moved G 21.0 mm to (2.03, 2.03)
- moved +9V 17.5 mm to (2.03, 4.57)
- moved JIN 3.07 mm to (2.03, 21.1)
- moved JOG 1.42 mm to (23.0, 18.5)
- moved SW2 0.63 mm to (12.7, 8.89)
- moved JIG 0.63 mm to (2.03, 18.5)
Connections:
- removed net IN: IN.1, SW2.A2
- removed net OUT: OUT.1, SW2.C3
- new net +9V: +9V.1, D1.C
- new net N$5: SW2.A2, U$1.1
- new net N$6: SW2.C3, U$1.5
- new net N$7: D1.A, U$1.3
- net GND: now also U$1.4
- net N$1: now also U$1.2; no longer LED.1
- net N$2: now also JOT.1; no longer JOUT.1
Routing:
- net OUT: track 20.6 -> 0.00 mm
- net N$6: track 0.00 -> 17.9 mm
- net N$1: track 34.0 -> 17.1 mm
- net IN: track 14.7 -> 0.00 mm
- net N$4: track 37.1 -> 50.5 mm
- net N$5: track 0.00 -> 13.3 mm
- net N$7: track 0.00 -> 12.2 mm
- net +9V: track 0.00 -> 3.17 mm
- net N$2: track 13.3 -> 15.1 mm
Other:
- board size 23.8 x 22.2 mm -> 25.1 x 23.5 mm
- board text added: "3PDT Daughterboard v1.2"
- board text added: "Xenocoder Designs 09 2018"
- board text removed: "3PDT Switch Jumper Board"
- board text removed: "Xenocoder Designs 01 2018"

Commit message: Update to panel with fixed Diode direction
Parts:
- D1: value 1N4001 -> (none)
- turned D1 to 270 degrees
Connections:
- net +9V: now also D1.A; no longer D1.C
- net N$7: now also D1.C; no longer D1.A
Other:
- board text added: "3PDT Daughterboard v1.3"
- board text added: "Xenocoder Designs 11 2018"
- board text removed: "3PDT Daughterboard v1.2"
- board text removed: "Xenocoder Designs 09 2018"
Changed lines of the file:
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@@
 <?xml version="1.0" encoding="utf-8"?>
 <!DOCTYPE eagle SYSTEM "eagle.dtd">
-<eagle version="9.1.0">
+<eagle version="9.2.2">
 <drawing>
 <settings>
@@
 <wire x1="25.07" y1="23.485" x2="0" y2="23.485" width="0" layer="20"/>
 <wire x1="0" y1="23.485" x2="0" y2="0" width="0" layer="20"/>
-<text x="21.971" y="1.27" size="0.8128" layer="25" font="vector" rot="R90">3PDT Daughterboard v1.2</text>
-<text x="23.495" y="1.27" size="0.8128" layer="25" font="vector" rot="R90">Xenocoder Designs 09 2018</text>
+<text x="21.971" y="1.27" size="0.8128" layer="25" font="vector" rot="R90">3PDT Daughterboard v1.3</text>
+<text x="23.495" y="1.27" size="0.8128" layer="25" font="vector" rot="R90">Xenocoder Designs 11 2018</text>
 </plain>
 <attributes>
@@
 <attribute name="NAME" x="4.445" y="3.81" size="1.016" layer="25" ratio="12" rot="R90"/>
 </element>
-<element name="D1" library="mb_diodes" package="DO41-3" value="1N4001" x="2.032" y="11.557" smashed="yes" rot="R90">
-<attribute name="NAME" x="2.667" y="10.4648" size="1.27" layer="25" ratio="12" rot="R90"/>
+<element name="D1" library="mb_diodes" package="DO41-3" value="" x="2.032" y="11.557" smashed="yes" rot="R270">
+<attribute name="NAME" x="1.397" y="12.6492" size="1.27" layer="25" ratio="12" rot="R270"/>
+<attribute name="VALUE" x="-0.762" y="13.462" size="1.27" layer="27" ratio="12" rot="R270"/>
 </element>
 </elements>
@@
 <wire x1="15.24" y1="6.35" x2="15.24" y2="17.399" width="0.4064" layer="16"/>
 </signal>
+<signal name="+9V">
+<contactref element="+9V" pad="1"/>
+<contactref element="D1" pad="A"/>
+<wire x1="2.032" y1="7.747" x2="2.032" y2="4.572" width="0.4064" layer="1"/>
+</signal>
 <signal name="N$7">
+<contactref element="D1" pad="C"/>
 <contactref element="U$1" pad="3"/>
-<contactref element="D1" pad="A"/>
-<wire x1="2.032" y1="15.367" x2="3.81" y2="17.145" width="0.4064" layer="1"/>
-<wire x1="3.81" y1="17.145" x2="9.906" y2="17.145" width="0.4064" layer="1"/>
-<wire x1="9.906" y1="17.145" x2="12.446" y2="19.685" width="0.4064" layer="1"/>
-</signal>
-<signal name="+9V">
-<contactref element="D1" pad="C"/>
-<contactref element="+9V" pad="1"/>
-<wire x1="2.032" y1="7.747" x2="2.032" y2="4.572" width="0.4064" layer="1"/>
+<wire x1="2.032" y1="15.367" x2="3.937" y2="15.367" width="0.4064" layer="1"/>
+<wire x1="3.937" y1="15.367" x2="6.35" y2="17.78" width="0.4064" layer="1"/>
+<wire x1="10.541" y1="17.78" x2="12.446" y2="19.685" width="0.4064" layer="1"/>
+<wire x1="6.35" y1="17.78" x2="10.541" y2="17.78" width="0.4064" layer="1"/>
 </signal>
 </signals>
