File: 3PDT Board.sch (EAGLE design)
At the start: 9 parts, among them SW2 3PDT

Commit message: Update to panel with fixed Diode direction
Parts:
- D1: value 1N4001 -> (none)
Connections:
- net +9V: now also D1.A; no longer D1.C
- net N$7: now also D1.C; no longer D1.A
Other:
- moved on the sheet: D1
Changed lines of the file:
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@@
 <?xml version="1.0" encoding="utf-8"?>
 <!DOCTYPE eagle SYSTEM "eagle.dtd">
-<eagle version="9.2.0">
+<eagle version="9.2.2">
 <drawing>
 <settings>
@@
 <part name="U$1" library="xc_library" deviceset="BOARDLINK" device=""/>
 <part name="+9V" library="mb_supply" deviceset="+9V(T)" device=""/>
-<part name="D1" library="mb_diodes" deviceset="1N400X" device=".3" value="1N4001"/>
+<part name="D1" library="mb_diodes" deviceset="1N400X" device=".3"/>
 </parts>
 <sheets>
@@
 </plain>
 <instances>
-<instance part="G" gate="GND" x="25.4" y="12.7">
+<instance part="G" gate="GND" x="25.4" y="12.7" smashed="yes">
 <attribute name="VALUE" x="23.495" y="9.525" size="1.778" layer="96"/>
 </instance>
-<instance part="JOG" gate="GND" x="20.32" y="15.24">
+<instance part="JOG" gate="GND" x="20.32" y="15.24" smashed="yes">
 <attribute name="VALUE" x="18.415" y="12.065" size="1.778" layer="96"/>
 </instance>
-<instance part="JOT" gate="G$1" x="38.1" y="12.7" rot="R270">
+<instance part="JOT" gate="G$1" x="38.1" y="12.7" smashed="yes" rot="R270">
 <attribute name="NAME" x="40.64" y="12.7" size="1.778" layer="95" rot="R270"/>
 </instance>
-<instance part="JIN" gate="G$1" x="15.24" y="38.1" rot="R90">
+<instance part="JIN" gate="G$1" x="15.24" y="38.1" smashed="yes" rot="R90">
 <attribute name="NAME" x="12.7" y="38.1" size="1.778" layer="95" rot="R90"/>
 </instance>
-<instance part="JIG" gate="GND" x="35.56" y="38.1">
+<instance part="JIG" gate="GND" x="35.56" y="38.1" smashed="yes">
 <attribute name="VALUE" x="37.973" y="36.703" size="1.778" layer="96"/>
 </instance>
-<instance part="SW2" gate="A" x="12.7" y="27.94">
+<instance part="SW2" gate="A" x="12.7" y="27.94" smashed="yes">
 <attribute name="NAME" x="8.255" y="20.193" size="1.778" layer="95" rot="R90"/>
 </instance>
-<instance part="SW2" gate="B" x="25.4" y="27.94">
+<instance part="SW2" gate="B" x="25.4" y="27.94" smashed="yes">
 <attribute name="NAME" x="20.955" y="20.193" size="1.778" layer="95" rot="R90"/>
 </instance>
-<instance part="SW2" gate="C" x="38.1" y="20.32">
+<instance part="SW2" gate="C" x="38.1" y="20.32" smashed="yes">
 <attribute name="NAME" x="33.655" y="12.573" size="1.778" layer="95" rot="R90"/>
 </instance>
-<instance part="U$1" gate="G$1" x="27.94" y="45.72">
+<instance part="U$1" gate="G$1" x="27.94" y="45.72" smashed="yes">
 <attribute name="NAME" x="26.924" y="53.34" size="1.778" layer="95"/>
 <attribute name="VALUE" x="39.878" y="47.752" size="1.778" layer="96"/>
 </instance>
-<instance part="+9V" gate="+9V" x="45.72" y="30.48" rot="R270">
+<instance part="+9V" gate="+9V" x="45.72" y="30.48" smashed="yes" rot="R270">
 <attribute name="VALUE" x="48.895" y="32.385" size="1.778" layer="96" rot="R270"/>
 </instance>
-<instance part="D1" gate="1" x="38.1" y="30.48">
-<attribute name="NAME" x="34.544" y="32.4866" size="1.778" layer="95" font="vector"/>
-<attribute name="VALUE" x="33.782" y="26.8986" size="1.778" layer="96" font="vector"/>
+<instance part="D1" gate="1" x="35.56" y="30.48" smashed="yes" rot="R180">
+<attribute name="NAME" x="39.116" y="28.4734" size="1.778" layer="95" font="vector" rot="R180"/>
+<attribute name="VALUE" x="39.878" y="34.0614" size="1.778" layer="96" font="vector" rot="R180"/>
 </instance>
 </instances>
@@
 </segment>
 </net>
+<net name="+9V" class="0">
+<segment>
+<pinref part="+9V" gate="+9V" pin="+9V"/>
+<pinref part="D1" gate="1" pin="A"/>
+<wire x1="43.18" y1="30.48" x2="40.64" y2="30.48" width="0.1524" layer="91"/>
+</segment>
+</net>
 <net name="N$7" class="0">
 <segment>
+<pinref part="D1" gate="1" pin="C"/>
 <pinref part="U$1" gate="G$1" pin="+9V"/>
-<pinref part="D1" gate="1" pin="A"/>
-<wire x1="33.02" y1="41.656" x2="33.02" y2="30.48" width="0.1524" layer="91"/>
-</segment>
-</net>
-<net name="+9V" class="0">
-<segment>
-<pinref part="D1" gate="1" pin="C"/>
-<pinref part="+9V" gate="+9V" pin="+9V"/>
-<wire x1="40.64" y1="30.48" x2="43.18" y2="30.48" width="0.1524" layer="91"/>
-</segment>
-</net>
+<wire x1="33.02" y1="30.48" x2="33.02" y2="41.656" width="0.1524" layer="91"/>
+</segment>
+</net>
